File: custom_microcontroller.sch (KiCad schematic (older format))
At the start: 29 parts, among them J1 Conn_01x05_Male, J2 Conn_01x02_Male, J3 Conn_01x08_Male, J4 Conn_01x02_Male, J5 Conn_01x02_Male, J6 Conn_01x06_Male, J7 Conn_01x02_Male, U1 NCP1117ST33T3G, U2 STM32F042G6Ux, U3 SN65HVD233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

Commit message: pcb smt assembly
Parts:
- C1, C10, C9: value 100nF -> 0.1uF; lcsc (none) -> C49678
- C11, C5: lcsc (none) -> C1779
- C12, C8: lcsc (none) -> C28323
- C2, C3: lcsc (none) -> C1792
- C4, C7: lcsc (none) -> C7171
- C6: lcsc (none) -> C1710
- D1, D2: lcsc (none) -> C2293
- R1, R2: lcsc (none) -> C17714
- R3: lcsc (none) -> C17590
- R4: lcsc (none) -> C17437
- U1: lcsc (none) -> C26537
- U3: lcsc (none) -> C61643
- Y1: lcsc (none) -> C90906
Changed lines of the file:
@@
 P 3500 7000
 F 0 "C10" H 3615 7046 50  0000 L CNN
-F 1 "100nF" H 3615 6955 50  0000 L CNN
+F 1 "0.1uF" H 3615 6955 50  0000 L CNN
 F 2 "Capacitor_SMD:C_0805_2012Metric_Pad1.15x1.40mm_HandSolder" H 3538 6850 50  0001 C CNN
 F 3 "~" H 3500 7000 50  0001 C CNN
+F 4 "C49678" H 3500 7000 50  0001 C CNN "lcsc"
 	1    3500 7000
 	1    0    0    -1
@@
 P 3000 7000
 F 0 "C9" H 3115 7046 50  0000 L CNN
-F 1 "100nF" H 3115 6955 50  0000 L CNN
+F 1 "0.1uF" H 3115 6955 50  0000 L CNN
 F 2 "Capacitor_SMD:C_0805_2012Metric_Pad1.15x1.40mm_HandSolder" H 3038 6850 50  0001 C CNN
 F 3 "~" H 3000 7000 50  0001 C CNN
+F 4 "C49678" H 3000 7000 50  0001 C CNN "lcsc"
 	1    3000 7000
 	1    0    0    -1
@@
 F 2 "Capacitor_SMD:C_0805_2012Metric_Pad1.15x1.40mm_HandSolder" H 4038 6850 50  0001 C CNN
 F 3 "~" H 4000 7000 50  0001 C CNN
+F 4 "C1779" H 4000 7000 50  0001 C CNN "lcsc"
 	1    4000 7000
 	1    0    0    -1
@@
 P 800 7000
 F 0 "C1" H 915 7046 50  0000 L CNN
-F 1 "100nF" H 915 6955 50  0000 L CNN
+F 1 "0.1uF" H 915 6955 50  0000 L CNN
 F 2 "Capacitor_SMD:C_0805_2012Metric_Pad1.15x1.40mm_HandSolder" H 838 6850 50  0001 C CNN
 F 3 "~" H 800 7000 50  0001 C CNN
+F 4 "C49678" H 800 7000 50  0001 C CNN "lcsc"
 	1    800  7000
 	1    0    0    -1
@@
 F 2 "Capacitor_SMD:C_0805_2012Metric_Pad1.15x1.40mm_HandSolder" H 1338 6850 50  0001 C CNN
 F 3 "~" H 1300 7000 50  0001 C CNN
+F 4 "C1779" H 1300 7000 50  0001 C CNN "lcsc"
 	1    1300 7000
 	1    0    0    -1
@@
 F 2 "Capacitor_SMD:C_0805_2012Metric_Pad1.15x1.40mm_HandSolder" H 1888 6850 50  0001 C CNN
 F 3 "~" H 1850 7000 50  0001 C CNN
+F 4 "C1710" H 1850 7000 50  0001 C CNN "lcsc"
 	1    1850 7000
 	1    0    0    -1
@@
 F 2 "Capacitor_SMD:C_0805_2012Metric_Pad1.15x1.40mm_HandSolder" H 2388 6850 50  0001 C CNN
 F 3 "~" H 2350 7000 50  0001 C CNN
+F 4 "C28323" H 2350 7000 50  0001 C CNN "lcsc"
 	1    2350 7000
 	1    0    0    -1
@@
 F 11 "ON Semiconductor" H 1850 6200 60  0001 L CNN "Manufacturer"
 F 12 "Active" H 1850 6300 60  0001 L CNN "Status"
+F 13 "C26537" H 1650 5100 50  0001 C CNN "lcsc"
 	1    1650 5100
 	1    0    0    -1
@@
 F 2 "Capacitor_Tantalum_SMD:CP_EIA-3216-18_Kemet-A_Pad1.58x1.35mm_HandSolder" H 1138 5400 50  0001 C CNN
 F 3 "~" H 1100 5550 50  0001 C CNN
+F 4 "C7171" H 1100 5550 50  0001 C CNN "lcsc"
 	1    1100 5550
 	1    0    0    -1
@@
 F 2 "Capacitor_Tantalum_SMD:CP_EIA-3216-18_Kemet-A_Pad1.58x1.35mm_HandSolder" H 2388 5400 50  0001 C CNN
 F 3 "~" H 2350 5550 50  0001 C CNN
+F 4 "C7171" H 2350 5550 50  0001 C CNN "lcsc"
 	1    2350 5550
 	1    0    0    -1
@@
 F 2 "LED_SMD:LED_0805_2012Metric_Pad1.15x1.40mm_HandSolder" H 3150 5650 50  0001 C CNN
 F 3 "~" H 3150 5650 50  0001 C CNN
+F 4 "C2293" H 3150 5650 50  0001 C CNN "lcsc"
 	1    3150 5650
 	0    -1   -1   0
@@
 F 2 "Resistor_SMD:R_0805_2012Metric_Pad1.15x1.40mm_HandSolder" V 3080 5300 50  0001 C CNN
 F 3 "~" H 3150 5300 50  0001 C CNN
+F 4 "C17590" H 3150 5300 50  0001 C CNN "lcsc"
 	1    3150 5300
 	1    0    0    -1
@@
 F 2 "LED_SMD:LED_0805_2012Metric_Pad1.15x1.40mm_HandSolder" H 850 1550 50  0001 C CNN
 F 3 "~" H 850 1550 50  0001 C CNN
+F 4 "C2293" H 850 1550 50  0001 C CNN "lcsc"
 	1    850  1550
 	0    -1   -1   0
@@
 F 2 "Resistor_SMD:R_0805_2012Metric_Pad1.15x1.40mm_HandSolder" V 780 2000 50  0001 C CNN
 F 3 "~" H 850 2000 50  0001 C CNN
+F 4 "C17714" H 850 2000 50  0001 C CNN "lcsc"
 	1    850  2000
 	-1   0    0    1
@@
 F 2 "Package_SO:SOIC-8_3.9x4.9mm_P1.27mm" H 2100 1100 50  0001 C CNN
 F 3 "http://www.ti.com/lit/ds/symlink/sn65hvd234.pdf" H 2000 2000 50  0001 C CNN
+F 4 "C61643" H 2100 1600 50  0001 C CNN "lcsc"
 	1    2100 1600
 	1    0    0    -1
@@
 F 2 "Capacitor_SMD:C_0805_2012Metric_Pad1.15x1.40mm_HandSolder" H 3338 1500 50  0001 C CNN
 F 3 "~" H 3300 1650 50  0001 C CNN
+F 4 "C28323" H 3300 1650 50  0001 C CNN "lcsc"
 	1    3300 1650
 	1    0    0    -1
@@
 F 2 "Crystal:Crystal_SMD_3225-4Pin_3.2x2.5mm_HandSoldering" H 1800 3600 50  0001 C CNN
 F 3 "~" H 1800 3600 50  0001 C CNN
+F 4 "C90906" H 1800 3600 50  0001 C CNN "lcsc"
 	1    1800 3600
 	0    -1   1    0
@@
 F 2 "Resistor_SMD:R_0805_2012Metric_Pad1.15x1.40mm_HandSolder" V 2480 3900 50  0001 C CNN
 F 3 "~" H 2550 3900 50  0001 C CNN
+F 4 "C17714" H 2550 3900 50  0001 C CNN "lcsc"
 	1    2550 3900
 	0    1    1    0
@@
 F 2 "Capacitor_SMD:C_0805_2012Metric_Pad1.15x1.40mm_HandSolder" H 1138 3750 50  0001 C CNN
 F 3 "~" H 1100 3900 50  0001 C CNN
+F 4 "C1792" H 1100 3900 50  0001 C CNN "lcsc"
 	1    1100 3900
 	0    1    1    0
@@
 F 2 "Capacitor_SMD:C_0805_2012Metric_Pad1.15x1.40mm_HandSolder" H 1138 3150 50  0001 C CNN
 F 3 "~" H 1100 3300 50  0001 C CNN
+F 4 "C1792" H 1100 3300 50  0001 C CNN "lcsc"
 	1    1100 3300
 	0    1    1    0
@@
 F 2 "Resistor_SMD:R_0805_2012Metric_Pad1.15x1.40mm_HandSolder" V 2630 1650 50  0001 C CNN
 F 3 "~" H 2700 1650 50  0001 C CNN
+F 4 "C17437" H 2700 1650 50  0001 C CNN "lcsc"
 	1    2700 1650
 	-1   0    0    1
